Commit message: Update launch files

File: source/hermes_description/urdf/hermes_parameters.xacro (robot description, xacro)
@@ -2,10 +2,10 @@
 <robot name="hermes" xmlns:xacro="http://www.ros.org/wiki/xacro">
     <!-- CHASSIS PARAMETERS -->
-    <xacro:property name="chassis_width" value="0.3" />
-    <xacro:property name="chassis_length" value="0.4" />
-    <xacro:property name="chassis_height" value="0.15" />
+    <xacro:property name="chassis_width" value="0.275" />
+    <xacro:property name="chassis_length" value="0.36" />
+    <xacro:property name="chassis_height" value="0.11" />
     <!-- WHEEL PARAMETERS -->
-    <xacro:property name="wheel_radius" value="0.05" />
-    <xacro:property name="wheel_length" value="0.03" />
+    <xacro:property name="wheel_radius" value="0.052" />
+    <xacro:property name="wheel_length" value="0.05" />
     <!--MASSES IN KG-->
     <xacro:property name="wheel_mass" value="0.08" />
