Commit message: Move from gazebo control to ROS2 control

File: source/hermes_description/urdf/hermes.urdf.xacro (robot description, xacro)
@@ -3,6 +3,6 @@
     <xacro:include filename="hermes_core.xacro" />
     <xacro:include filename="hermes.gazebo" />
-    <xacro:include filename="gazebo_control.xacro" />
-    <!-- <xacro:include filename="ros2_control.xacro" /> -->
+    <!-- <xacro:include filename="gazebo_control.xacro" /> -->
+    <xacro:include filename="ros2_control.xacro" />
     <xacro:include filename="lidar.xacro" />
     <xacro:include filename="camera.xacro" />

File: source/hermes_description/urdf/ros2_control.xacro (robot description, xacro)
@@ -3,6 +3,22 @@
     <ros2_control name="GazeboSystem" type="system">
         <hardware>
-            <plugin>
+            <plugin>gz_ros2_control/GazeboSimSystem</plugin>
         </hardware>
+        <joint name="left_middle_wheel_joint">
+            <command_interface name="velocity">
+                <param name="min">-10</param>
+                <param name="max">10</param>
+            </command_interface>
+            <state_interface name="velocity" />
+            <state_interface name="position" />
+        </joint>
+        <joint name="right_middle_wheel_joint">
+            <command_interface name="velocity">
+                <param name="min">-10</param>
+                <param name="max">10</param>
+            </command_interface>
+            <state_interface name="velocity" />
+            <state_interface name="position" />
+        </joint>
     </ros2_control>
 </robot>

Commit message: configured to work with ros2_control

File: source/hermes_description/urdf/hermes.urdf.xacro (robot description, xacro)
@@ -2,11 +2,14 @@
 <robot name="hermes" xmlns:xacro="http://www.ros.org/wiki/xacro">
     <!-- Use Gazebo or not -->
-    <xacro:arg name="use_gazebo" default="true" />
+    <xacro:arg name="use_gazebo" default="false" />
     <!-- Use mock components or not? Note: If using mock, must disable gazebo -->
     <xacro:arg name="use_mock" default="false" />
     <!-- Actual Hardware -->
-    <xacro:arg name="use_hardware" default="false" />
+    <xacro:arg name="use_hardware" default="true" />
     <!-- Use ros2_control or not? -->
     <xacro:arg name="use_ros2_control" default="true" />
+    <!-- my controllers parameters yaml file-->
+    <xacro:property name="controllers_yaml" value="$(find hermes_description)/config/my_controllers.yaml" />
+    <xacro:property name="controllers_config" value="${xacro.load_yaml(controllers_yaml)}" />
     <xacro:include filename="hermes_core.xacro" />
     <xacro:include filename="hermes.gazebo" />

File: source/hermes_description/urdf/ros2_control.xacro (robot description, xacro)
@@ -18,4 +18,7 @@
                 <param name="example_param_hw_stop_duration_sec">0</param>
                 <param name="serial_port">/dev/ttyACM0</param>
+                <param name="baud_rate">115200</param>
+                <param name="loop_rate">${controllers_config['controller_manager']['ros__parameters']['update_rate']}</param> <!-- 100Hz -->
+                <param name="timeout_ms">1000</param> <!-- 1 second -->
              </xacro:if>
         </hardware>
