Commit message: Fix xacro file

File: source/hermes_description/urdf/lidar.xacro (robot description, xacro)
@@ -3,8 +3,8 @@
     <joint name="laser_joint" type="fixed">
         <parent link="chassis" />
-        <child link="laser_frame" />
+        <child link="ldlidar_link" />
         <origin xyz="0.1 0 ${chassis_height}" rpy="0 0 0"/>
     </joint>
-    <link name="laser_frame">
+    <link name="ldlidar_link">
         <visual>
             <geometry>
@@ -22,9 +22,9 @@
         </xacro:inertial_cylinder>
     </link>
-    <gazebo reference="laser_frame">
+    <gazebo reference="ldlidar_link">
         <!-- A scanning lidar ray-->
         <sensor name="laser" type="gpu_lidar">
             <!-- Origin of the virtual sensor -->
-            <pose relative_to="lidar_frame"> 0 0 0 0 0 0 </pose>
+            <pose relative_to="ldlidar_link"> 0 0 0 0 0 0 </pose>
             <topic>scan</topic>
             <visualize>false</visualize>

Commit message: lidar

File: source/hermes_description/urdf/lidar.xacro (robot description, xacro)
@@ -6,5 +6,5 @@
         <origin xyz="0.1 0 ${chassis_height}" rpy="0 0 0"/>
     </joint>
-    <link name="ldlidar_link">
+    <!-- <link name="ldlidar_base">
         <visual>
             <geometry>
@@ -21,5 +21,22 @@
             <origin xyz="0 0 0" rpy="0 0 0" />
         </xacro:inertial_cylinder>
+    </link> -->
+    <link name="ldlidar_base">
+        <visual>
+            <origin xyz="0 0 0" rpy="0 0 0"/>
+            <geometry>
+                <mesh filename="package://ldlidar_node/urdf/model/LD19.stl" scale="0.001 0.001 0.001" />
+            </geometry>
+            <material name="ldlidar_mat">
+                <color rgba="0.8 0.8 0.8 0.8"/>
+            </material>
+        </visual>
     </link>
+    <joint name="ldlidar_link_joint" type="fixed">
+        <parent link="ldlidar_base"/>
+        <child link="ldlidar_link"/>
+        <origin xyz="0 0 0.02745" rpy="0 0 0" />
+    </joint>
+    <link name="ldlidar_link" />
     <gazebo reference="ldlidar_link">
         <!-- A scanning lidar ray-->

Commit message: fix urdf

File: source/hermes_description/urdf/lidar.xacro (robot description, xacro)
@@ -6,5 +6,5 @@
         <origin xyz="0.1 0 ${chassis_height}" rpy="0 0 0"/>
     </joint>
-    <!-- <link name="ldlidar_base">
+    <link name="ldlidar_base">
         <visual>
             <geometry>
@@ -21,6 +21,6 @@
             <origin xyz="0 0 0" rpy="0 0 0" />
         </xacro:inertial_cylinder>
-    </link> -->
-    <link name="ldlidar_base">
+    </link>
+    <!-- <link name="ldlidar_base">
         <visual>
             <origin xyz="0 0 0" rpy="0 0 0"/>
@@ -32,11 +32,11 @@
             </material>
         </visual>
-    </link>
-    <joint name="ldlidar_link_joint" type="fixed">
+    </link> -->
+    <!-- <joint name="ldlidar_link_joint" type="fixed">
         <parent link="ldlidar_base"/>
         <child link="ldlidar_link"/>
         <origin xyz="0 0 0.02745" rpy="0 0 0" />
     </joint>
-    <link name="ldlidar_link" />
+    <link name="ldlidar_link" /> -->
     <gazebo reference="ldlidar_link">
         <!-- A scanning lidar ray-->

Commit message: fixed naming issue with link

File: source/hermes_description/urdf/lidar.xacro (robot description, xacro)
@@ -6,5 +6,5 @@
         <origin xyz="0.1 0 ${chassis_height}" rpy="0 0 0"/>
     </joint>
-    <link name="ldlidar_base">
+    <link name="ldlidar_link">
         <visual>
             <geometry>
